Commit message: We can now spawn a sphere in Gazebo
Using "rosrun gazebo_ros spawn_model" service. We will integrate this into tumor_generation shortly.

File: catkin_ws/src/ck_robot/urdf/sphere.urdf (robot description, URDF)
Before this commit: robot tumor, 1 links, 0 joints
Links:
- link base_link: mass None -> 1.0; geometry visual sphere radius=0.1
