Commit message: Greatly reduced mass in CK_robot URDF and created URDF for sphere

File: catkin_ws/src/ck_robot/urdf/ck_robot.urdf (robot description, URDF)
Before this commit: robot ck_robot, 8 links, 7 joints
Links:
- link base_link: mass 60.1875042918917 -> 1E-5
- link link_1: mass 1 -> 1E-5
- link link_2: mass 1 -> 1E-5
- link link_3: mass 1 -> 1E-5
- link link_4: mass 1 -> 1E-5
- link link_5: mass 1 -> 1E-5
- link link_6: mass 1 -> 1E-5

Commit message: Changed home position of the robot

File: catkin_ws/src/ck_robot/urdf/ck_robot.urdf (robot description, URDF)
Before this commit: robot ck_robot, 8 links, 7 joints
Joints:
- joint joint_1: origin xyz=0.268464971217371 -0.598518951650115 0.442083103301491 rpy=1.5707963267949 0 0.144460400809996 -> xyz=0.268464971217371 -0.598518951650115 0.442083103301491 rpy=1.5707963267949 0 -0.00605138749237428
- joint joint_2: origin xyz=0.285 0.279 0 rpy=0 0 -1.27141640789434 -> xyz=0.285 0.279 0 rpy=0 0 -1.53895939549721
- joint joint_3: origin xyz=0 0.67999999999999 0 rpy=-3.14159265358979 0 -0.313045625626455 -> xyz=0 0.67999999999999 0 rpy=3.14159265358979 0 -1.5859187836385
- joint joint_4: origin xyz=-0.474166946244357 -0.022499999999998 0.0329999999999995 rpy=0 0.956127472462032 1.5707963267949 -> xyz=-0.474166946244357 -0.022499999999998 0.0329999999999995 rpy=3.14159265358978 -1.48381066723595 -1.57079632679489
- joint joint_5: origin xyz=0 0.192333053755625 0 rpy=2.51840109391516 0 3.14159265358979 -> xyz=0 0.192333053755625 0 rpy=-1.64879993389354 0 0
- joint joint_6: origin xyz=-0.0159999999999946 0 0 rpy=0 0 0.232084976469764 -> xyz=-0.0159999999999946 0 0 rpy=0 0 -0.889895608487581
