Commit message: global frame fix

File: ck_robot/urdf/ck_robot.urdf (robot description, URDF)
Before this commit: robot ck_robot, 7 links, 6 joints
Links:
- link link_1: mass 15.0344590133941 -> 15.0344818329302
- link link_2: mass 13.9289336493322 -> 13.7581112963571
- link link_3: mass 13.027483798185 -> 13.0275184665504
- link link_4: mass 2.38078149447115 -> 2.38079036358208
- link link_5: mass 1.7928112729056 -> 1.79281371541231
- link link_6: mass 24.8877788431059 -> 24.8877693978715
Joints:
- joint joint_1: origin xyz=0.268464971217371 -0.598518951650115 0.442083103301491 rpy=1.5707963267949 0 0.144460400809996 -> xyz=-0.00383300568916015 0.00270725046410668 0.340050258271999 rpy=1.5707963267949 0 -0.00605138749237428
- joint joint_2: origin xyz=0.285 0.279 0 rpy=0 0 -1.27141640789434 -> xyz=0.285 0.279 0.0600067744860645 rpy=0 0 -1.53895939549721
- joint joint_3: origin xyz=0 0.67999999999999 0 rpy=-3.14159265358979 0 -0.313045625626455 -> xyz=0 0.680000000000004 0 rpy=3.14159265358979 0 -1.5859187836385
- joint joint_4: origin xyz=-0.474166946244357 -0.022499999999998 0.0329999999999995 rpy=0 0.956127472462032 1.5707963267949 -> xyz=-0.473242791686348 -0.0224999999999999 0.0930067744860649 rpy=3.14159265358978 -1.48381066723595 -1.57079632679489
- joint joint_5: origin xyz=0 0.192333053755625 0 rpy=2.51840109391516 0 3.14159265358979 -> xyz=0 0.193257208313652 0 rpy=-1.64879993389354 0 0
- joint joint_6: origin xyz=-0.0159999999999946 0 0 rpy=0 0 0.232084976469764 -> xyz=-0.00299999999999894 0 0.102405955386691 rpy=0 0 -0.889895608487581
